File: StackZ80Kicad/SRAM_Maskable.kicad_sch (KiCad schematic)
At the start: 14 parts, among them SW5 SW_DIP_x08, SW6 SW_DIP_x08, SW7 SW_DIP_x08, SW8 SW_DIP_x08, SW9 Enable_BT, U10 74LS32, U7 28C256, U8 74HCT688, U9 74HCT688

Commit message: Add files via upload
Parts:
- removed U7: 28C256, symbol Memory_EEPROM:28C256
- added U15: CY62256-70PC, Package_DIP:DIP-28_W15.24mm, symbol Memory_RAM:CY62256-70PC
- renumbered D6 to D7, RN2 to RN6, RN4 to RN7, RN3 to RN8, RN5 to RN9, SW5 to SW10, SW7 to SW11, SW6 to SW12, SW8 to SW13, SW9 to SW14, U10 to U12, U8 to U13, U9 to U14
Connections:
- net 5V: now also U15.28 (VCC)
- net ADDR0: now also U15.10 (A0)
- net ADDR1: now also U15.9 (A1)
- net ADDR10: now also U15.21 (A10)
- net ADDR11: now also U15.23 (A11)
- net ADDR12: now also U15.2 (A12)
- net ADDR13: now also U15.26 (A13)
- net ADDR14: now also U15.1 (A14)
- net ADDR2: now also U15.8 (A2)
- net ADDR3: now also U15.7 (A3)
- net ADDR4: now also U15.6 (A4)
- net ADDR5: now also U15.5 (A5)
- net ADDR6: now also U15.4 (A6)
- net ADDR7: now also U15.3 (A7)
- net ADDR8: now also U15.25 (A8)
- net ADDR9: now also U15.24 (A9)
- net DATA0: now also U15.11 (Q0)
- net DATA1: now also U15.12 (Q1)
- net DATA2: now also U15.13 (Q2)
- net DATA3: now also U15.15 (Q3)
- net DATA4: now also U15.16 (Q4)
- net DATA5: now also U15.17 (Q5)
- net DATA6: now also U15.18 (Q6)
- net DATA7: now also U15.19 (Q7)
- net GND: now also U15.14 (GND)
- net ~{CS}: now also U15.20 (~{CS})
- net ~{OE}: now also U15.22 (~{OE})
- net ~{WE}: now also U15.27 (~{WE})
