File: StackZ80Kicad/PowerModule.kicad_sch (KiCad schematic)
At the start: 10 parts, among them J1 Main USB Power and Serial, J2 Another USB Power and Serial, J3 Conn_01x20_Pin, J4 Conn_01x20_Pin, SW1 Power Switch, U1 CH340C, U2 CH340C(CH2), U3 Z84C20, U4 74HCT688_Serial1Comp

Commit message: Add files via upload
Parts:
- removed J3, J4: Conn_01x20_Pin, symbol Connector:Conn_01x20_Pin
- removed U3: Z84C20, Package_DIP:DIP-40_W15.24mm, symbol Interface:Z84C20
- added C1, C3, C4, C5: C104, symbol Device:C
- added C2: C_100uF_Power, symbol Device:C_Polarized
- added D1: Power LED, symbol Device:LED
- added D2: TX_1, symbol Device:LED
- added D3: RX_1, symbol Device:LED
- added D4: TX_2, symbol Device:LED
- added D5: RX_2, symbol Device:LED
- added R1, R7, R8, R9: 5.1kOhm_Resistor_USB_C, symbol Device:R
- added R2, R3, R4, R5, R6: 1k_Resistor_LED, symbol Device:R
- added RN1: Address_PullUP, Resistor_THT:R_Array_SIP7, symbol Device:R_Network06
- added SW2: Address_Program_DIP, symbol Switch:SW_DIP_x06
- added SW3: IEI Switch, symbol Switch:SW_Push_SPDT
- added U5: Z84C42BB6, Package_DIP:DIP-40_W15.24mm, symbol PCM_Z80_ST:Z84C42BB6
- F1: value Polyfuse for Power -> 3A Polyfuse for Power
Connections:
- net Addr2: now also U4.6 (P2); no longer U4.2 (P0)
- net Addr3: now also U4.8 (P3); no longer U4.4 (P1)
- net Addr4: now also U4.11 (P4); no longer U4.6 (P2)
- net Addr5: now also U4.13 (P5); no longer U4.8 (P3)
- net Addr6: now also U4.15 (P6); no longer U4.11 (P4)
- net Addr7: now also U4.17 (P7); no longer U4.13 (P5)
- net GND: now reaches J2.A1 (GND), J2.A12 (GND), J2.B1 (GND), J2.B12 (GND)
- net GND: now also J1.A1 (GND), J1.A12 (GND), J1.B1 (GND), J1.B12 (GND), J1.SH (SHIELD), J2.SH (SHIELD), U1.1 (GND), U1.15 (R232), U2.1 (GND), U2.15 (R232), U4.2 (P0), U4.3 (R0), U4.4 (P1), U4.5 (R1), C1.2, C2.2, C3.2, C4.2, D1.1 (K), D2.1 (K), D3.1 (K), D4.1 (K), D5.1 (K), R1.2, R7.2, R8.2, R9.2, U5.19 (~{DCDA}), U5.22 (~{DCDB}), U5.31 (GND)
- net at J2.A4 (VBUS), J2.A9 (VBUS), J2.B4 (VBUS)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: now also F1.2, J1.A4 (VBUS), J1.A9 (VBUS), J1.B4 (VBUS), J1.B9 (VBUS)
- net at J2.A5 (CC1): now also R7.1
- net at J2.A6 (D+): now also J2.B6 (D+), U2.5 (UD+)
- net at J2.A7 (D-): now also J2.B7 (D-), U2.6 (UD-)
- net at J2.B5 (CC2): now also R1.1
- net ~{RTSB}: now reaches U2.14 (~{RTS})
- net ~{RTSB}: now also U5.24 (~{RTSB})
- net 5V: now reaches U2.16 (VCC)
- net 5V: now also SW1.1 (A), U1.16 (VCC), U4.20 (VCC), C1.1, C2.1, C3.1, C4.1, C5.1, R2.2, SW3.3 (C), U5.9 (V_{CC})
- net Tx_2: now reaches U2.2 (TXD)
- net Tx_2: now also R5.2, U5.29 (RxDB)
- net Rx_2: now reaches U2.3 (RXD)
- net Rx_2: now also R6.2, U5.26 (TxDB)
- net ~{CTSB}: now reaches U2.9 (~{CTS})
- net ~{CTSB}: now also U5.23 (~{CTSB})
- net at F1.1: now also SW1.2 (B)
- net at J1.A5 (CC1): now also R8.1
- net at J1.A6 (D+): now also J1.B6 (D+), U1.5 (UD+)
- net at J1.A7 (D-): now also J1.B7 (D-), U1.6 (UD-)
- net at J1.B5 (CC2): now also R9.1
- net ~{RTSA}: now reaches U1.14 (~{RTS})
- net ~{RTSA}: now also U5.17 (~{RTSA})
- net Tx_1: now reaches U1.2 (TXD)
- net Tx_1: now also R3.2, U5.12 (RxDA)
- net Rx_1: now reaches U1.3 (RXD)
- net Rx_1: now also R4.2, U5.15 (TxDA)
- net ~{CTSA}: now reaches U1.9 (~{CTS})
- net ~{CTSA}: now also U5.18 (~{CTSA})
- net ~{IORQ}: now reaches U4.1 (G)
- net ~{IORQ}: now also U5.36 (~{IORQ})
- net at U4.10 (GND): now also C5.2, SW2.10, SW2.11, SW2.12, SW2.7, SW2.8, SW2.9
- net at U4.12 (R4): now also RN1.5 (R4), SW2.3
- net at U4.14 (R5): now also RN1.4 (R3), SW2.4
- net at U4.16 (R6): now also RN1.3 (R2), SW2.5
- net at U4.18 (R7): now also RN1.2 (R1), SW2.6
- net ~{SIO_CS}: now reaches U4.19 (P=R)
- net ~{SIO_CS}: now also U5.35 (~{CE})
- net at U4.7 (R2): now also RN1.7 (R6), SW2.1
- net at U4.9 (R3): now also RN1.6 (R5), SW2.2
- new net: D1.2 (A), R2.1
- new net: D2.2 (A), R4.1
- new net: D3.2 (A), R3.1
- new net: D4.2 (A), R6.1
- new net: SW3.2 (B), U5.6 (IEI)
- new net: U5.13 (~{RxCA}), U5.14 (~{TxCA}), U5.27 (~{TxCB}), U5.28 (~{RxCB})
- new net: D5.2 (A), R5.1
- new net Addr0: U5.34 (B/~{A})
- new net Addr1: U5.33 (C/~{D})
- new net CLK: U5.20 (CLK)
- new net Data0: U5.40 (D_{0})
- new net Data1: U5.1 (D_{1})
- new net Data2: U5.39 (D_{2})
- new net Data3: U5.2 (D_{3})
- new net Data4: U5.38 (D_{4})
- new net Data5: U5.3 (D_{5})
- new net Data6: U5.37 (D_{6})
- new net Data7: U5.4 (D_{7})
- new net IEDown: U5.7 (IEO)
- new net IEUp: SW3.1 (A)
- new net ~{INT}: U5.5 (~{INT})
- new net ~{M1}: U5.8 (~{M1})
- new net ~{RD}: U5.32 (~{RD})
- new net ~{RESET}: U5.21 (~{RESET})
- no-connect marks 0 -> 18
Other:
- note removed: "5V GND TX1 RX1 TX2 RX2"
- note removed: "📋 Layer 0：電源與雙串口模組完整元件清單 (BOM)1. 核心與介面晶片 (IC Chips)1x Zilog SIO/2 晶片 (型號：Z84C4006PEC 或 Z84C4010PEC)封裝： DIP-40 (直插式，建議搭配 40-pin IC 座)用途： Z80 專用的雙通道序列通訊控制器。2x USB-to-UART 晶片 (型號：CH340C -- 注意尾碼必須是 C)封裝： SOP-16 (表面黏著)用途： 將 USB 訊號轉為 TTL 序列訊號（免外接晶振）。1x 地址解碼晶片 (型號：74HCT138 或 74HCT30)封裝： DIP-16 (直插) 或 SOIC-16 (表面黏著)用途： 讓 Z80 CPU 能夠精確定位這片板子的 I/O 位置。2. 連接器與開關 (Connectors & Switches)2x USB-C 插座 (KiCad 推薦型號：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"
- moved on the sheet: F1, U1, U2, U4

Commit message: Add files via upload
Other:
- note added: "ALERT THE IE UP DOWN SYSTEM IS REPLACED BY 30 INT Pins BUT THIS PART IS NOT YET UPDATED"
Changed lines of the file:
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@@
 	(generator_version "10.0")
 	(paper "A4")
+	(text "ALERT\nTHE IE UP DOWN SYSTEM IS REPLACED BY 30 INT Pins BUT THIS PART IS NOT YET UPDATED"
+		(exclude_from_sim no)
+		(at 98.425 110.49 0)
+		(effects
+			(font
+				(size 1.27 1.27)
+			)
+		)
+	)
 	(junction
 		(at 53.34 45.72)
