File: StackZ80Kicad/Control_Panel.kicad_sch (KiCad schematic)
At the start: 8 parts

Commit message: Add files via upload
Parts:
- added BAR10, BAR11: Signal LEDs, Display:HDSP-4830, symbol LED:HDSP-4830_2
- added D9: Address_Check, symbol Device:LED
- added R15: 5.1kOhm_Resistor_PullUp, symbol Device:R
- added RN11, RN13: R_10Kohm_PullUP, Resistor_THT:R_Array_SIP9, symbol Device:R_Network08
- added SW16, SW18: Wait, symbol Switch:SW_SPDT
- added SW17, SW19: SW_DIP_x08, symbol Switch:SW_DIP_x08
- added U11: 4013, symbol 4xxx:4013
- added U16: 74HC244, symbol 74xx:74HC244
- added U17, U18: 74HCT688, symbol 74xx:74HCT688
Connections:
- net 5V: now also D9.1 (K), R15.1, SW17.1, SW17.2, SW17.3, SW17.4, SW17.5, SW17.6, SW17.7, SW17.8, SW19.1, SW19.2, SW19.3, SW19.4, SW19.5, SW19.6, SW19.7, SW19.8, U11.14 (VDD), U17.20 (VCC), U18.20 (VCC)
- net CLK: now also U11.1 (Q), U11.11 (C)
- net GND: now also BAR10.13 (K), BAR10.14 (K), BAR10.15 (K), BAR10.16 (K), BAR10.17 (K), BAR10.18 (K), BAR10.19 (K), BAR10.20 (K), BAR11.13 (K), BAR11.14 (K), BAR11.15 (K), BAR11.16 (K), BAR11.17 (K), BAR11.18 (K), BAR11.19 (K), BAR11.20 (K), RN11.1 (common), RN13.1 (common), SW16.1 (A), SW18.1 (A), U11.3 (C), U11.5 (D), U11.7 (VSS), U17.1 (G), U17.10 (GND), U18.1 (G), U18.10 (GND)
- net ~{BUSREQ}: now also SW18.2 (B)
- net ~{WAIT}: now also SW16.2 (B), U11.13 (Q)
- new net: BAR11.5 (A), RN13.6 (R5), SW19.12, U18.12 (R4)
- new net: BAR11.6 (A), RN13.7 (R6), SW19.11, U18.14 (R5)
- new net: BAR11.7 (A), RN13.8 (R7), SW19.10, U18.16 (R6)
- new net: BAR11.8 (A), RN13.9 (R8), SW19.9, U18.18 (R7)
- new net: D9.2 (A), U11.9 (D), U17.19 (P=R), U18.19 (P=R)
- new net: BAR11.1 (A), RN13.2 (R1), SW19.16, U18.3 (R0)
- new net: BAR11.2 (A), RN13.3 (R2), SW19.15, U18.5 (R1)
- new net: BAR11.3 (A), RN13.4 (R3), SW19.14, U18.7 (R2)
- new net: BAR11.4 (A), RN13.5 (R4), SW19.13, U18.9 (R3)
- new net: R15.2, U11.6 (S)
- new net: BAR10.7 (A), RN11.8 (R7), SW17.10, U17.16 (R6)
- new net: BAR10.6 (A), RN11.7 (R6), SW17.11, U17.14 (R5)
- new net: BAR10.5 (A), RN11.6 (R5), SW17.12, U17.12 (R4)
- new net: BAR10.4 (A), RN11.5 (R4), SW17.13, U17.9 (R3)
- new net: BAR10.3 (A), RN11.4 (R3), SW17.14, U17.7 (R2)
- new net: BAR10.2 (A), RN11.3 (R2), SW17.15, U17.5 (R1)
- new net: BAR10.1 (A), RN11.2 (R1), SW17.16, U17.3 (R0)
- new net: BAR10.8 (A), RN11.9 (R8), SW17.9, U17.18 (R7)
- new net ADDR0: U17.2 (P0)
- new net ADDR1: U17.4 (P1)
- new net ADDR10: U18.6 (P2)
- new net ADDR11: U18.8 (P3)
- new net ADDR12: U18.11 (P4)
- new net ADDR13: U18.13 (P5)
- new net ADDR14: U18.15 (P6)
- new net ADDR15: U18.17 (P7)
- new net ADDR2: U17.6 (P2)
- new net ADDR3: U17.8 (P3)
- new net ADDR4: U17.11 (P4)
- new net ADDR5: U17.13 (P5)
- new net ADDR6: U17.15 (P6)
- new net ADDR7: U17.17 (P7)
- new net ADDR8: U18.2 (P0)
- new net ADDR9: U18.4 (P1)
Other:
- moved on the sheet: BAR1, BAR5
