File: StackZ80Kicad/EEPROM_Maskable.kicad_sch (KiCad schematic)
At the start: 14 parts, among them SW5 SW_DIP_x08, SW6 SW_DIP_x08, SW7 SW_DIP_x08, SW8 SW_DIP_x08, SW9 Enable_BT, U10 74LS32, U7 28C256, U8 74HCT688, U9 74HCT688

Commit message: Add files via upload
Changed lines of the file:
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@@
-		)
-	)
-	(label "ADDR[0..15]"
-		(at 57.15 38.1 0)
-		(effects
-			(font
-				(size 1.27 1.27)
-			)
-			(justify left bottom)
 		)
 	)
@@
 		)
 	)
+	(hierarchical_label "ADDR[0..15]"
+		(shape bidirectional)
+		(at 57.15 38.1 0)
+		(effects
+			(font
+				(size 1.27 1.27)
+			)
+			(justify left)
+		)
+	)
