File: StackZ80Kicad/Minimum.kicad_sch (KiCad schematic)
At the start: 59 parts, among them J3 Conn_01x24_Pin, J4 Conn_01x16_Pin, U19 CY62256-70PC, U20 28C256, U21 74LS573, U22 74LS573, U23 74LS573, U24 74LS573, U26 Z84C0010P, U27 74AHCT1G04

Commit message: Add files via upload
Parts:
- removed R16, R17, R18, R19, R20, R21, R22, R23, R24, R25, R26, R27, R28, R29, R30, R31, R32, R33, R34, R35, R36, R37, R38, R39, R40, R41, R42, R43, R44, R45, R46, R47, R48, R49, R50, R51, R52, R53: 1k, symbol Device:R
- added RN10, RN12, RN14, RN15, RN16: 1k_Resistor_Network, Resistor_THT:R_Array_SIP9, symbol Device:R_Network08
- C10: footprint (none) -> PCM_Capacitor_THT_AKL:C_Disc_D4.3mm_W1.9mm_P5.00mm
- J3: footprint (none) -> Connector_PinHeader_2.54mm:PinHeader_1x24_P2.54mm_Vertical
- J4: footprint (none) -> Connector_PinHeader_2.54mm:PinHeader_1x16_P2.54mm_Vertical
- R54, R55, R56, R57, R58: footprint (none) -> Resistor_THT:R_Axial_DIN0207_L6.3mm_D2.5mm_P7.62mm_Horizontal
- U20: footprint (none) -> Package_DIP:DIP-28_W15.24mm
- U21, U22, U23, U24: footprint (none) -> Package_DIP:DIP-20_W7.62mm
- U27: footprint (none) -> Package_TO_SOT_SMD:SOT-23-5_HandSoldering
Connections:
- net 5V: now also RN15.1 (common), RN16.1 (common)
- net CLK: now also BAR14.20 (K); no longer BAR13.16 (K)
- net DATA0: now also BAR13.1 (A); no longer BAR12.7 (A)
- net DATA1: now also BAR13.2 (A); no longer BAR12.8 (A)
- net DATA2: now also BAR13.3 (A); no longer BAR12.9 (A)
- net DATA3: now also BAR13.4 (A); no longer BAR12.10 (A)
- net DATA4: now also BAR13.5 (A); no longer BAR13.1 (A)
- net DATA5: now also BAR13.6 (A); no longer BAR13.2 (A)
- net DATA6: now also BAR13.7 (A); no longer BAR13.3 (A)
- net DATA7: now also BAR13.8 (A); no longer BAR13.4 (A)
- net GND: now also RN10.1 (common), RN12.1 (common), RN14.1 (common)
- net ~{BUSACK}: now also BAR12.13 (K); no longer BAR14.18 (K)
- net ~{BUSREQ}: now also BAR12.14 (K); no longer BAR14.19 (K)
- net ~{HALT}: now also BAR14.13 (K); no longer BAR14.15 (K)
- net ~{INT}: now also BAR12.12 (K); no longer BAR14.17 (K)
- net ~{IORQ}: now also BAR14.17 (K); no longer BAR13.13 (K)
- net ~{M1}: now also BAR14.19 (K); no longer BAR13.15 (K)
- net ~{MREQ}: now also BAR14.18 (K); no longer BAR13.14 (K)
- net ~{NMI}: now also BAR12.11 (K), R55.2; no longer BAR14.16 (K)
- net ~{RD}: now also BAR14.16 (K); no longer BAR13.12 (K)
- net ~{RESET}: now also BAR14.11 (K); no longer BAR14.13 (K)
- net ~{RFSH}: now also BAR14.14 (K); no longer BAR14.20 (K)
- net ~{WAIT}: now also BAR14.12 (K); no longer BAR14.14 (K)
- net ~{WR}: now also BAR14.15 (K); no longer BAR13.11 (K)
- net at BAR14.5 (A): now also RN15.7 (R6)
- net at BAR13.10 (A): now also RN16.4 (R3)
- net at BAR13.17 (K): now also RN14.5 (R4)
- net at BAR13.18 (K): now also RN14.4 (R3)
- net at BAR13.19 (K): now also RN14.3 (R2)
- net at BAR13.20 (K): now also RN14.2 (R1)
- net at BAR13.9 (A): now also RN16.5 (R4)
- net at BAR14.3 (A): now also RN15.9 (R8)
- net at BAR12.18 (K): now also RN12.6 (R5)
- net at BAR9.12 (K): now also RN12.2 (R1)
- net at BAR14.4 (A): now also RN15.8 (R7)
- net at BAR14.7 (A): now also RN15.5 (R4)
- net at BAR14.1 (A): now also RN16.3 (R2)
- net at BAR14.10 (A): now also RN15.2 (R1)
- net at BAR14.2 (A): now also RN16.2 (R1)
- net at BAR14.6 (A): now also RN15.6 (R5)
- net at BAR14.8 (A): now also RN15.4 (R3)
- net at BAR14.9 (A): now also RN15.3 (R2)
- net at BAR9.20 (K): now also RN10.2 (R1)
- net at BAR12.17 (K): now also RN12.7 (R6)
- net at BAR12.15 (K): now also RN12.9 (R8)
- net at BAR9.18 (K): now also RN10.4 (R3)
- net at BAR9.14 (K): now also RN10.8 (R7)
- net at BAR9.11 (K): now also RN12.3 (R2)
- net at BAR12.16 (K): now also RN12.8 (R7)
- net at BAR12.19 (K): now also RN12.5 (R4)
- net at BAR12.20 (K): now also RN12.4 (R3)
- net at BAR9.13 (K): now also RN10.9 (R8)
- net at BAR9.15 (K): now also RN10.7 (R6)
- net at BAR9.16 (K): now also RN10.6 (R5)
- net at BAR9.17 (K): now also RN10.5 (R4)
- net at BAR9.19 (K): now also RN10.3 (R2)
- new net: BAR12.10 (A), RN16.6 (R5)
- new net: BAR12.9 (A), RN16.7 (R6)
- new net: BAR12.8 (A), RN16.8 (R7)
- new net: BAR12.7 (A), RN16.9 (R8)
- new net: BAR13.16 (K), RN14.6 (R5)
- new net: BAR13.15 (K), RN14.7 (R6)
- new net: BAR13.14 (K), RN14.8 (R7)
- new net: BAR13.13 (K), RN14.9 (R8)
